File: eagle/star.brd (EAGLE design)
At the start: 40 x 40 mm, 30 parts, among them IC1 TINY13V-10MM0

Commit message: small code updates, cleanup
Parts:
- BT1: value (none) -> 3V
- C1: value (none) -> 100n
- R1: value (none) -> 68
- moved BT1 0.50 mm to (20.0, 16.0)
- turned LED1 to 0 degrees
- turned LED10 to 292.5 degrees
- turned LED11 to 22.5 degrees
- turned LED12 to 337.5 degrees
- turned LED13 to 202.5 degrees
- turned LED14 to 112.5 degrees
- turned LED15 to 67.5 degrees
- turned LED16 to 157.5 degrees
- turned LED2 to 90 degrees
- turned LED3 to 180 degrees
- turned LED4 to 270 degrees
- turned LED5 to 45 degrees
- turned LED6 to 135 degrees
- turned LED7 to 225 degrees
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Connections:
- removed net N$1: LED10.C, LED11.C, LED12.C, LED13.C, LED14.C, LED15.C, LED16.C, LED9.C, R1.1
- new net RES: LED10.A, LED11.A, LED12.A, LED13.A, LED14.A, LED15.A, LED16.A, LED9.A, R1.2
- net 3V: now also R1.1; no longer R1.2
- net GND: now also LED1.C, LED10.C, LED11.C, LED12.C, LED13.C, LED14.C, LED15.C, LED16.C, LED2.C, LED3.C, LED4.C, LED5.C, LED6.C, LED7.C, LED8.C, LED9.C; no longer LED1.A, LED10.A, LED11.A, LED12.A, LED13.A, LED14.A, LED15.A, LED16.A, LED2.A, LED3.A, LED4.A, LED5.A, LED6.A, LED7.A, LED8.A, LED9.A
- net MISO: now also LED1.A, LED2.A, LED3.A, LED4.A; no longer LED1.C, LED2.C, LED3.C, LED4.C
- net MOSI: now also LED5.A, LED6.A, LED7.A, LED8.A; no longer LED5.C, LED6.C, LED7.C, LED8.C
Routing:
- net N$1: track 35.7 -> 0.00 mm, vias 1 -> 0
- net RES: track 0.00 -> 35.7 mm, vias 0 -> 1
