File: eagle/star.sch (EAGLE design)
At the start: 30 parts, among them IC1 TINY13V-10MM0

Commit message: small code updates, cleanup
Parts:
- BT1: value (none) -> 3V
- C1: value (none) -> 100n
- R1: value (none) -> 68
Connections:
- removed net N$1: LED10.C, LED11.C, LED12.C, LED13.C, LED14.C, LED15.C, LED16.C, LED9.C, R1.1
- new net RES: LED10.A, LED11.A, LED12.A, LED13.A, LED14.A, LED15.A, LED16.A, LED9.A, R1.2
- net 3V: now also R1.1; no longer R1.2
- net GND: now also LED1.C, LED10.C, LED11.C, LED12.C, LED13.C, LED14.C, LED15.C, LED16.C, LED2.C, LED3.C, LED4.C, LED5.C, LED6.C, LED7.C, LED8.C, LED9.C; no longer LED1.A, LED10.A, LED11.A, LED12.A, LED13.A, LED14.A, LED15.A, LED16.A, LED2.A, LED3.A, LED4.A, LED5.A, LED6.A, LED7.A, LED8.A, LED9.A
- net MISO: now also LED1.A, LED2.A, LED3.A, LED4.A; no longer LED1.C, LED2.C, LED3.C, LED4.C
- net MOSI: now also LED5.A, LED6.A, LED7.A, LED8.A; no longer LED5.C, LED6.C, LED7.C, LED8.C
Other:
- note added: "*Adjust this value according to your LEDs"
- note added: "Purple LEDs"
- note added: "White LEDs"
- note added: "Yellow LEDs"
- moved on the sheet: BT1, LED5, LED6, LED7, LED8, PAD1, PAD2, PAD3, PAD4, R1
